Commit message: removed fixed, zero-mass joints and links

File: aliengo_env/urdf/aliengo_original.urdf (robot description, URDF)
Before this commit: robot aliengo_description, 17 links, 16 joints
Links:
- added link base; visual box size=0.001 0.001 0.001
- added link imu_link, mass 0.001; collision box size=.001 .001 .001; visual box size=0.001 0.001 0.001
Joints:
- added joint floating_base: type fixed, parent base, child trunk, origin xyz=0 0 0 rpy=0 0 0
- added joint imu_joint: type fixed, parent trunk, child imu_link, origin xyz=0 0 0 rpy=0 0 0
